File: 05_CADs/02_ElectronicDesign_EDA/KiCad/BD-SMD_PD/BD-SMD_PD.kicad_pcb (KiCad board)
At the start: 2 copper layers, 190 x 130 mm, 210 parts, among them J1 Conn_01x02_sens, J10 Conn_01x02_sens, J11 Conn_01x02_heater, J12 Conn_01x02_heater, J13 Conn_01x02_sens, J14 Conn_01x02_sens, J15 Conn_01x02_heater, J16 Conn_01x02_heater, J17 Conn_01x02_sens, J18 Conn_01x02_sens, J19 Conn_01x02_heater, J2 Conn_01x02_sens, J20 Conn_01x02_heater, J21 Conn_01x02_sens, J22 Conn_01x02_sens, J23 Conn_01x02_heater, J24 Conn_01x02_heater, J25 Conn_01x02_sens, J26 Conn_01x02_sens, J27 Conn_01x02_heater, J28 Conn_01x02_heater, J29 Conn_01x02_sens, J3 Conn_01x02_heater, J30 Conn_01x02_sens, J31 Conn_01x02_heater, J32 Conn_01x02_heater, J33 Conn_01x02_sens, J34 Conn_01x02_sens, J35 Conn_01x02_heater, J36 Conn_01x02_heater, J37 Conn_01x02_sens, J38 Conn_01x02_sens, J39 Conn_01x02_heater, J4 Conn_01x02_heater, J40 Conn_01x02_heater, J41 Conn_01x02_sens, J42 Conn_01x02_sens, J43 Conn_01x02_heater, J44 Conn_01x02_heater, J45 Conn_01x02_sens, J46 Conn_01x02_sens, J47 Conn_01x02_heater, J48 Conn_01x02_heater, J49 Conn_01x09, J5 Conn_01x02_sens, J50 Conn_01x03, J6 Conn_01x02_sens, J7 Conn_01x02_heater, J8 Conn_01x02_heater, J9 Conn_01x02_sens, Q1 DMG3418L, Q10 DMG3418L, Q11 DMG3418L, Q12 DMG3418L, Q13 DMG3418L, Q14 DMG3418L, Q15 DMG3418L, Q16 DMG3418L, Q17 DMG3418L, Q18 DMG3418L, Q19 DMG3418L, Q2 DMG3418L, Q20 DMG3418L, Q21 DMG3418L, Q22 DMG3418L, Q23 DMG3418L, Q24 DMG3418L, Q3 DMG3418L, Q4 DMG3418L, Q5 DMG3418L, Q6 DMG3418L, Q7 DMG3418L, Q8 DMG3418L, Q9 DMG3418L, U1 ADS7028, U2 ADS7028, U3 ADS7028, U4 ADS7028, U5 ADS7028, U6 ADS7028

Commit message: Production files created
Parts:
- R12, R24, R36, R48, R60, R72: footprint Capacitor_SMD:C_0603_1608Metric_Pad1.08x0.95mm_HandSolder -> Resistor_SMD:R_0402_1005Metric_Pad0.72x0.64mm_HandSolder
Other:
- outline, holes or cut-outs redrawn
