File: 05_CADs/02_ElectronicDesign_EDA/KiCad/BD-SMD_PD/BD-SMD_PD.kicad_sch (KiCad schematic)
At the start: 2 parts, among them J49 Conn_01x09, J50 Conn_01x03

Commit message: mods
Parts:
- J49: LCSC (none) -> C379029
- J50: LCSC (none) -> C2882762
Changed lines of the file:
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@@
+      (effects (font (size 1.27 1.27)) hide)
+    )
+    (property "LCSC" "C379029" (id 4) (at 248.92 90.17 0)
       (effects (font (size 1.27 1.27)) hide)
     )
@@
       (effects (font (size 1.27 1.27)) hide)
     )
-    (property "LCSC" "" (id 4) (at 248.92 111.76 0)
+    (property "LCSC" "C2882762" (id 4) (at 248.92 111.76 0)
       (effects (font (size 1.27 1.27)) hide)
     )
