File: 05_CADs/02_ElectronicDesign_EDA/KiCad/BD-SMD_PD/unit0.kicad_sch (KiCad schematic)
At the start: 29 parts, among them J1 Conn_01x02_sens, J2 Conn_01x02_sens, J3 Conn_01x02_heater, J4 Conn_01x02_heater, J5 Conn_01x02_sens, J6 Conn_01x02_sens, J7 Conn_01x02_heater, J8 Conn_01x02_heater, Q1 DMG3418L, Q2 DMG3418L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

Commit message: Production files created
Parts:
- C1: LCSC (none) -> C77404
- C2: LCSC (none) -> C393685
- J1, J3: LCSC (none) -> C189893
- Q1: LCSC (none) -> C151026
- R1: LCSC (none) -> C5119777
- R12: footprint Capacitor_SMD:C_0603_1608Metric_Pad1.08x0.95mm_HandSolder -> Resistor_SMD:R_0402_1005Metric_Pad0.72x0.64mm_HandSolder
- R3: LCSC (none) -> C705665
- R5: LCSC (none) -> C2763769
- U1: LCSC (none) -> C880341
Changed lines of the file:
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@@
     (property "Reference" "R12" (id 0) (at 123.19 144.78 90))
     (property "Value" "100k" (id 1) (at 123.19 147.32 90))
-    (property "Footprint" "Capacitor_SMD:C_0603_1608Metric_Pad1.08x0.95mm_HandSolder" (id 2) (at 124.46 144.018 90)
+    (property "Footprint" "Resistor_SMD:R_0402_1005Metric_Pad0.72x0.64mm_HandSolder" (id 2) (at 124.46 144.018 90)
       (effects (font (size 1.27 1.27)) hide)
     )
@@
       (effects (font (size 1.27 1.27)) (justify left) hide)
     )
+    (property "LCSC" " C151026" (id 4) (at 50.8 60.96 0)
+      (effects (font (size 1.27 1.27)) hide)
+    )
     (pin "1")
     (pin "2")
@@
     )
     (property "Datasheet" "~" (id 3) (at 213.36 31.75 0)
+      (effects (font (size 1.27 1.27)) hide)
+    )
+    (property "LCSC" "C77404" (id 4) (at 213.36 31.75 0)
       (effects (font (size 1.27 1.27)) hide)
     )
@@
       (effects (font (size 1.27 1.27)) hide)
     )
+    (property "LCSC" "C2763769" (id 4) (at 48.26 67.31 90)
+      (effects (font (size 1.27 1.27)) hide)
+    )
     (pin "1")
     (pin "2")
@@
     )
     (property "Datasheet" "~" (id 3) (at 223.52 31.75 0)
+      (effects (font (size 1.27 1.27)) hide)
+    )
+    (property "LCSC" "C393685" (id 4) (at 223.52 31.75 0)
       (effects (font (size 1.27 1.27)) hide)
     )
@@
     )
     (property "Datasheet" "https://www.ti.com/lit/ds/symlink/ads7028.pdf" (id 3) (at 223.52 114.3 0)
+      (effects (font (size 1.27 1.27)) hide)
+    )
+    (property "LCSC" "C880341" (id 4) (at 223.52 77.47 0)
       (effects (font (size 1.27 1.27)) hide)
     )
@@
       (effects (font (size 1.27 1.27)) hide)
     )
+    (property "LCSC" "C705665" (id 4) (at 38.1 60.96 90)
+      (effects (font (size 1.27 1.27)) hide)
+    )
     (pin "1")
     (pin "2")
@@
       (effects (font (size 1.27 1.27)) hide)
     )
+    (property "LCSC" "C5119777" (id 4) (at 44.45 30.48 90)
+      (effects (font (size 1.27 1.27)) hide)
+    )
     (pin "1")
     (pin "2")
@@
     )
     (property "Datasheet" "~" (id 3) (at 59.69 30.48 0)
+      (effects (font (size 1.27 1.27)) hide)
+    )
+    (property "LCSC" "C189893" (id 4) (at 59.69 30.48 0)
       (effects (font (size 1.27 1.27)) hide)
     )
@@
       (effects (font (size 1.27 1.27)) hide)
     )
+    (property "LCSC" "C189893" (id 4) (at 59.69 52.07 0)
+      (effects (font (size 1.27 1.27)) hide)
+    )

Commit message: mods
Parts:
- C2: LCSC C393685 -> C180354
- C3: LCSC (none) -> C180354
- C4: LCSC (none) -> C77404
- J2, J4, J5, J6, J7, J8: LCSC (none) -> C189893
- Q2, Q3, Q4: LCSC (none) -> C151026
- R1: LCSC C5119777 -> C513708
- R10, R4, R9: LCSC (none) -> C705665
- R11, R12, R6: LCSC (none) -> C2142686
- R2, R7, R8: LCSC (none) -> C513708
- R5: LCSC C2763769 -> C2142686
Changed lines of the file:
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@@
+      (effects (font (size 1.27 1.27)) hide)
+    )
+    (property "LCSC" "C2142686" (id 4) (at 124.46 142.24 0)
       (effects (font (size 1.27 1.27)) hide)
     )
@@
     )
     (property "Datasheet" "~" (id 3) (at 120.65 105.41 0)
+      (effects (font (size 1.27 1.27)) hide)
+    )
+    (property "LCSC" "C513708" (id 4) (at 120.65 105.41 0)
       (effects (font (size 1.27 1.27)) hide)
     )
@@
       (effects (font (size 1.27 1.27)) hide)
     )
-    (property "LCSC" "C2763769" (id 4) (at 48.26 67.31 90)
+    (property "LCSC" "C2142686" (id 4) (at 48.26 67.31 90)
       (effects (font (size 1.27 1.27)) hide)
     )
@@
     )
     (property "Datasheet" "~" (id 3) (at 135.89 127 0)
+      (effects (font (size 1.27 1.27)) hide)
+    )
+    (property "LCSC" "C189893" (id 4) (at 135.89 127 0)
       (effects (font (size 1.27 1.27)) hide)
     )
@@
       (effects (font (size 1.27 1.27)) hide)
     )
+    (property "LCSC" "C705665" (id 4) (at 114.3 60.96 0)
+      (effects (font (size 1.27 1.27)) hide)
+    )
     (pin "1")
     (pin "2")
@@
       (effects (font (size 1.27 1.27)) hide)
     )
+    (property "LCSC" "C705665" (id 4) (at 38.1 135.89 0)
+      (effects (font (size 1.27 1.27)) hide)
+    )
     (pin "1")
     (pin "2")
@@
       (effects (font (size 1.27 1.27)) hide)
     )
-    (property "LCSC" "C393685" (id 4) (at 223.52 31.75 0)
+    (property "LCSC" "C180354" (id 4) (at 223.52 31.75 0)
       (effects (font (size 1.27 1.27)) hide)
     )
@@
     (property "Datasheet" "http://www.diodes.com/assets/Datasheets/DMG3418L.pdf" (id 3) (at 127 135.89 0)
       (effects (font (size 1.27 1.27)) (justify left) hide)
+    )
+    (property "LCSC" " C151026" (id 4) (at 127 135.89 0)
+      (effects (font (size 1.27 1.27)) hide)
     )
     (pin "1")
@@
       (effects (font (size 1.27 1.27)) hide)
     )
+    (property "LCSC" "C705665" (id 4) (at 114.3 135.89 0)
+      (effects (font (size 1.27 1.27)) hide)
+    )
     (pin "1")
     (pin "2")
@@
       (effects (font (size 1.27 1.27)) hide)
     )
+    (property "LCSC" "C189893" (id 4) (at 59.69 127 0)
+      (effects (font (size 1.27 1.27)) hide)
+    )
     (pin "1")
     (pin "2")
@@
       (effects (font (size 1.27 1.27)) hide)
     )
+    (property "LCSC" "C513708" (id 4) (at 44.45 105.41 0)
+      (effects (font (size 1.27 1.27)) hide)
+    )
     (pin "1")
     (pin "2")
@@
     )
     (property "Datasheet" "~" (id 3) (at 226.06 104.14 0)
+      (effects (font (size 1.27 1.27)) hide)
+    )
+    (property "LCSC" "C77404" (id 4) (at 226.06 104.14 0)
       (effects (font (size 1.27 1.27)) hide)
     )
@@
     (property "Datasheet" "http://www.diodes.com/assets/Datasheets/DMG3418L.pdf" (id 3) (at 50.8 135.89 0)
       (effects (font (size 1.27 1.27)) (justify left) hide)
+    )
+    (property "LCSC" " C151026" (id 4) (at 50.8 135.89 0)
+      (effects (font (size 1.27 1.27)) hide)
     )
     (pin "1")
@@
     )
     (property "Datasheet" "~" (id 3) (at 124.46 67.31 0)
+      (effects (font (size 1.27 1.27)) hide)
+    )
+    (property "LCSC" "C2142686" (id 4) (at 124.46 67.31 0)
       (effects (font (size 1.27 1.27)) hide)
     )
@@
       (effects (font (size 1.27 1.27)) hide)
     )
-    (property "LCSC" "C5119777" (id 4) (at 44.45 30.48 90)
+    (property "LCSC" "C513708" (id 4) (at 44.45 30.48 90)
       (effects (font (size 1.27 1.27)) hide)
     )
@@
       (effects (font (size 1.27 1.27)) (justify left) hide)
     )
+    (property "LCSC" " C151026" (id 4) (at 127 60.96 0)
+      (effects (font (size 1.27 1.27)) hide)
+    )
     (pin "1")
     (pin "2")
@@
     )
     (property "Datasheet" "~" (id 3) (at 135.89 52.07 0)
+      (effects (font (size 1.27 1.27)) hide)
+    )
+    (property "LCSC" "C189893" (id 4) (at 135.89 52.07 0)
       (effects (font (size 1.27 1.27)) hide)
     )
@@
     )
     (property "Datasheet" "~" (id 3) (at 135.89 105.41 0)
+      (effects (font (size 1.27 1.27)) hide)
+    )
+    (property "LCSC" "C189893" (id 4) (at 135.89 105.41 0)
       (effects (font (size 1.27 1.27)) hide)
     )
@@
     )
     (property "Datasheet" "~" (id 3) (at 120.65 30.48 0)
+      (effects (font (size 1.27 1.27)) hide)
+    )
+    (property "LCSC" "C513708" (id 4) (at 120.65 30.48 0)
       (effects (font (size 1.27 1.27)) hide)
     )
@@
       (effects (font (size 1.27 1.27)) hide)
     )
+    (property "LCSC" "C2142686" (id 4) (at 48.26 142.24 0)
+      (effects (font (size 1.27 1.27)) hide)
+    )
     (pin "1")
     (pin "2")
@@
       (effects (font (size 1.27 1.27)) hide)
     )
+    (property "LCSC" "C189893" (id 4) (at 59.69 105.41 0)
+      (effects (font (size 1.27 1.27)) hide)
+    )
     (pin "1")
     (pin "2")
@@
       (effects (font (size 1.27 1.27)) hide)
     )
+    (property "LCSC" "C180354" (id 4) (at 233.68 31.75 0)
+      (effects (font (size 1.27 1.27)) hide)
+    )
     (pin "1")
     (pin "2")
@@
       (effects (font (size 1.27 1.27)) hide)
     )
+    (property "LCSC" "C189893" (id 4) (at 135.89 30.48 0)
+      (effects (font (size 1.27 1.27)) hide)
+    )

Commit message: mods in bom
Parts:
- C1, C4: LCSC C77404 -> C77046
- C2, C3: LCSC C180354 -> C77055
- R11, R12, R5, R6: LCSC C2142686 -> C60491
Changed lines of the file:
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@@
       (effects (font (size 1.27 1.27)) hide)
     )
-    (property "LCSC" "C2142686" (id 4) (at 124.46 142.24 0)
+    (property "LCSC" "C60491" (id 4) (at 124.46 142.24 0)
       (effects (font (size 1.27 1.27)) hide)
     )
@@
       (effects (font (size 1.27 1.27)) hide)
     )
-    (property "LCSC" "C77404" (id 4) (at 213.36 31.75 0)
+    (property "LCSC" "C77046" (id 4) (at 213.36 31.75 0)
       (effects (font (size 1.27 1.27)) hide)
     )
@@
       (effects (font (size 1.27 1.27)) hide)
     )
-    (property "LCSC" "C2142686" (id 4) (at 48.26 67.31 90)
+    (property "LCSC" "C60491" (id 4) (at 48.26 67.31 90)
       (effects (font (size 1.27 1.27)) hide)
     )
@@
       (effects (font (size 1.27 1.27)) hide)
     )
-    (property "LCSC" "C180354" (id 4) (at 223.52 31.75 0)
+    (property "LCSC" "C77055" (id 4) (at 223.52 31.75 0)
       (effects (font (size 1.27 1.27)) hide)
     )
@@
       (effects (font (size 1.27 1.27)) hide)
     )
-    (property "LCSC" "C77404" (id 4) (at 226.06 104.14 0)
+    (property "LCSC" "C77046" (id 4) (at 226.06 104.14 0)
       (effects (font (size 1.27 1.27)) hide)
     )
@@
       (effects (font (size 1.27 1.27)) hide)
     )
-    (property "LCSC" "C2142686" (id 4) (at 124.46 67.31 0)
+    (property "LCSC" "C60491" (id 4) (at 124.46 67.31 0)
       (effects (font (size 1.27 1.27)) hide)
     )
@@
       (effects (font (size 1.27 1.27)) hide)
     )
-    (property "LCSC" "C2142686" (id 4) (at 48.26 142.24 0)
+    (property "LCSC" "C60491" (id 4) (at 48.26 142.24 0)
       (effects (font (size 1.27 1.27)) hide)
     )
@@
       (effects (font (size 1.27 1.27)) hide)
     )
-    (property "LCSC" "C180354" (id 4) (at 233.68 31.75 0)
-      (effects (font (size 1.27 1.27)) hide)
-    )
+    (property "LCSC" "C77055" (id 4) (at 233.68 31.75 0)
+      (effects (font (size 1.27 1.27)) hide)
+    )
